File: circuits/connectors_pcb/connectors.brd (EAGLE design)
At the start: 34.5 x 16 mm, 9 parts, among them J1 1x3 RA Female .1", J2 1x3 RA Female .1", Q2 SI2369DS-T1-GE3, U1 MIC5219 5V

Commit message: Minor updates to schematic and board files. Still UNTESTED
Parts:
- turned C2 to 90 degrees
Connections:
- net 5V: no longer Q2.1
- net GND: now also Q2.1
Routing:
- net 5V: track 20.0 -> 15.4 mm
- net GND: track 55.9 -> 60.4 mm
Changed lines of the file:
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@@
 </element>
 <element name="C1" library="rcl" package="C0402K" value="470p" x="18.5" y="4.9" rot="MR180"/>
-<element name="C2" library="rcl" package="C0603K" value="10u" x="22" y="4.5" rot="R270"/>
+<element name="C2" library="rcl" package="C0603K" value="10u" x="22" y="4.5" rot="R90"/>
 <element name="Q2" library="transistor-fet" package="SOT23" value="SI2369DS-T1-GE3" x="26.5" y="7"/>
 <element name="R1" library="rcl" package="R0603" value="10k" x="18.5" y="4.5" rot="R90"/>
@@
 <contactref element="C2" pad="2"/>
 <wire x1="18.5" y1="3.65" x2="18.5" y2="1.5" width="0.4064" layer="1"/>
-<wire x1="22" y1="3.625" x2="22" y2="1.5" width="0.4064" layer="1"/>
+<contactref element="Q2" pad="1"/>
+<wire x1="25.55" y1="5.9" x2="22" y2="5.9" width="0.4064" layer="1"/>
+<wire x1="22" y1="5.9" x2="20.375" y2="5.9" width="0.4064" layer="1"/>
+<wire x1="20.375" y1="5.9" x2="20.375" y2="4.9" width="0.4064" layer="1"/>
+<wire x1="22" y1="5.375" x2="22" y2="5.9" width="0.4064" layer="1"/>
 </signal>
 <signal name="5V">
@@
 <via x="25.81" y="3" extent="1-16" drill="0.5" shape="octagon"/>
 <contactref element="U$1" pad="4"/>
-<wire x1="25.81" y1="3" x2="16.3001" y2="3" width="0.4064" layer="16"/>
 <wire x1="25.81" y1="1.5" x2="25.81" y2="3" width="0.4064" layer="1"/>
-<contactref element="Q2" pad="1"/>
-<wire x1="25.81" y1="3" x2="23.25" y2="3" width="0.4064" layer="1"/>
-<wire x1="23.25" y1="3" x2="23.25" y2="5.375" width="0.4064" layer="1"/>
-<wire x1="25.55" y1="5.9" x2="23.25" y2="5.9" width="0.4064" layer="1"/>
+<wire x1="25.81" y1="3" x2="22" y2="3" width="0.4064" layer="1"/>
 <contactref element="C2" pad="1"/>
-<wire x1="22" y1="5.375" x2="23.25" y2="5.375" width="0.4064" layer="1"/>
-<wire x1="23.25" y1="5.375" x2="23.25" y2="5.9" width="0.4064" layer="1"/>
+<wire x1="22" y1="3" x2="22" y2="3.625" width="0.4064" layer="1"/>
+<wire x1="16.3001" y1="3" x2="25.81" y2="3" width="0.4064" layer="16"/>
 </signal>
 <signal name="DATA">
