File: circuits/connectors_pcb/connectors.sch (EAGLE design)
At the start: 9 parts, among them J1 1x3 RA Female .1", J2 1x3 RA Female .1", Q2 SI2369DS-T1-GE3, U1 MIC5219 5V

Commit message: Minor updates to schematic and board files. Still UNTESTED
Connections:
- net 5V: no longer Q2.G
- net GND: now also Q2.G
Other:
- note removed: "Compare signal for microcontroller board"
Changed lines of the file:
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@@
 <part name="GND5" library="SparkFun-Aesthetics" deviceset="GND" device=""/>
 <part name="Q2" library="transistor-fet" deviceset="SI2333DS" device="" value="SI2369DS-T1-GE3"/>
-<part name="SUPPLY7" library="SparkFun-Aesthetics" deviceset="5V" device=""/>
 <part name="R1" library="rcl" deviceset="R-EU_" device="R0603" value="10k"/>
 <part name="GND1" library="SparkFun-Aesthetics" deviceset="GND" device=""/>
@@
 <part name="GND7" library="SparkFun-Aesthetics" deviceset="GND" device=""/>
 <part name="SUPPLY8" library="SparkFun-Aesthetics" deviceset="5V" device=""/>
+<part name="GND8" library="SparkFun-Aesthetics" deviceset="GND" device=""/>
 </parts>
 <sheets>
 <sheet>
 <plain>
-<text x="43.18" y="63.5" size="1.778" layer="97">Compare signal for microcontroller board</text>
 </plain>
 <instances>
@@
 <instance part="GND5" gate="1" x="43.18" y="-5.08"/>
 <instance part="Q2" gate="G$1" x="5.08" y="53.34" rot="R90"/>
-<instance part="SUPPLY7" gate="G$1" x="7.62" y="40.64" rot="R180"/>
 <instance part="R1" gate="G$1" x="-2.54" y="45.72" rot="R90"/>
 <instance part="GND1" gate="1" x="-2.54" y="38.1"/>
@@
 <instance part="GND7" gate="1" x="63.5" y="38.1"/>
 <instance part="SUPPLY8" gate="G$1" x="63.5" y="55.88"/>
+<instance part="GND8" gate="1" x="7.62" y="38.1"/>
 </instances>
 <busses>
@@
 <wire x1="63.5" y1="43.18" x2="63.5" y2="40.64" width="0.1524" layer="91"/>
 </segment>
+<segment>
+<pinref part="Q2" gate="G$1" pin="G"/>
+<pinref part="GND8" gate="1" pin="GND"/>
+<wire x1="7.62" y1="40.64" x2="7.62" y2="48.26" width="0.1524" layer="91"/>
+</segment>
 </net>
 <net name="5V" class="0">
@@
 </segment>
 <segment>
-<wire x1="7.62" y1="40.64" x2="7.62" y2="48.26" width="0.1524" layer="91"/>
-<pinref part="Q2" gate="G$1" pin="G"/>
-<pinref part="SUPPLY7" gate="G$1" pin="5V"/>
-</segment>
-<segment>
